Commit message: Removed references to Gazebo.

File: src/jackal_ignition/models/jackal.urdf.xacro (robot description, xacro)
@@ -45,13 +45,4 @@
       </inertial>
     </link>
-    <gazebo reference="${prefix}_wheel_link">
-      <material>Gazebo/DarkGrey</material>
-      <selfCollide>false</selfCollide>
-      <mu1 value="0.5"/>
-      <mu2 value="0.5"/>
-      <kp value="10000000.0" />
-      <kd value="1" />
-      <fdir1 value="1 0 0"/>
-    </gazebo>
     <joint name="${prefix}_wheel" type="continuous">
       <parent link="chassis_link"/>
@@ -222,6 +213,4 @@
     <origin xyz="${mount_spacing} 0 0" />
   </joint>
-  <!-- Bring in simulation data for Gazebo. -->
-  <xacro:include filename="$(find jackal_description)/urdf/jackal.gazebo" />
   <!-- Optional standard accessories, including their simulation data. The rendering
        of these into the final description is controlled by optenv variables, which
